Commit message: 完成了简单的Sapien的抓取操作,尝试进行提交

File: description/ur_e_description/urdf/ur.gazebo.xacro (robot description, xacro)
@@ -29,6 +29,6 @@
       <kinematic>0</kinematic>
       <gravity>1</gravity>
-      <!--<mu>1</mu>-->
-      <mu2>1</mu2>
+      <mu>2000</mu>
+      <mu2>1000</mu2>
       <fdir1>0 0 0</fdir1>
       <!--<slip1>0</slip1>

File: sapien_simulator/urdf/ur5e.urdf (robot description, URDF)
Before this commit: robot ur5e, 31 links, 30 joints
Links:
- added link robotiq_2f_85_ee_link
Joints:
- added joint robotiq_ur_coupler_robotiq_2f_85_ee_joint: type fixed, parent robotiq_arg2f_base_link, child robotiq_2f_85_ee_link, origin xyz=0 0 0.1493 rpy=0 0 0
