Commit message: 完成了Gazebo和Sapien的坐标系对应,从而分割图能正确生成

File: sapien_simulator/urdf/ur5e_origin.urdf (robot description, URDF)
Before this commit: robot ur5e, 32 links, 31 joints
Joints:
- joint table_joint: child base_link -> table; origin xyz=0 -0.24 0.0 rpy=0.0 0.0 0 -> xyz=0.0 0.0 -0.005 rpy=0.0 0.0 -1.57079; parent table -> world
- joint world_joint: child table -> base_link; origin xyz=0.0 0.0 -0.005 rpy=0.0 0.0 -1.57 -> xyz=-0.24 -0.005 0 rpy=0.0 0.0 -1.57079
